Commit message: added gazebo files

File: bot_description/urdf/bot.xacro (robot description, xacro)
@@ -84,11 +84,11 @@
   </collision>
 </link>
-<joint name="Revolute 1" type="continuous">
+<joint name="Revolute1" type="continuous">
   <origin xyz="0.0 -0.1 0.06" rpy="0 0 0"/>
   <parent link="base_link"/>
   <child link="right_wheel_1"/>
-  <axis xyz="0.0 -1.0 0.0"/>
+  <axis xyz="0.0 1.0 0.0"/>
 </joint>
-<joint name="Revolute 2" type="continuous">
+<joint name="Revolute2" type="continuous">
   <origin xyz="0.0 0.1 0.06" rpy="0 0 0"/>
   <parent link="base_link"/>
